File: buck-converter-real.kicad_sch (KiCad schematic)
At the start: 55 parts, among them J1 BOOT, J2 XT60, J3 Battery out (3V6-4V2) NiMH 3S, J4 POWER, J5 UART 2, J6 DM3CS-SF, J7 UART 1, J8 I2C, J9 SWD, Q1 Q_NMOS_DGS, Q2 CSD18540Q5B - 60-V, Q3 Q_PMOS_DGS, U1 AP2112K-3.3 (3V3 LDO), U5 LM5109BMA (Mosfet Driver), U6 AS78L12RTR-G1 (12V LDO)

Commit message: Update layout - after successful board test
Parts:
- removed J1: BOOT, Connector_PinHeader_2.54mm:PinHeader_1x03_P2.54mm_Vertical, symbol Connector_Generic:Conn_01x03
- removed J8: I2C, Connector_PinHeader_2.54mm:PinHeader_1x04_P2.54mm_Vertical, symbol Connector_Generic:Conn_01x04
- added J1: USB_C_Receptacle_USB2.0_16P, Connector_USB:USB_C_Receptacle_G-Switch_GT-USB-7010ASV, symbol Connector:USB_C_Receptacle_USB2.0_16P
- added J10, J11: JST_01x04, Connectors_JST:JST_SH_SM04B-SRSS-TB_04x1.00mm_Angled, symbol Connector_Generic:Conn_01x04
- D3: footprint PCM_Diode_SMD_AKL:D_SMC -> Diode_SMD:D_SMA
- L2: footprint Inductor_SMD:L_10.4x10.4_H4.8 -> buck-forest:L_10.4x10.4_H4.8
- U6: value AS78L12RTR-G1 (12V LDO) -> 78L12L (12V LDO) (35V max); footprint OptoDevice:Broadcom_APDS-9160-003 -> Package_TO_SOT_SMD:SOT-89-3
- renumbered USBC to USBC1
Connections:
- net +3.3V: now also J10.3 (Pin_3)
- net GND: now also J10.4 (Pin_4)
- net I2C-SCL: now also J10.1 (Pin_1)
- net I2C-SDA: now also J10.2 (Pin_2)
- net BOOT renamed VSENSE_VOUT
- new net: J1.A1 (GND), J1.A12 (GND), J1.B1 (GND), J1.B12 (GND)
- new net: J1.A4 (VBUS), J1.A9 (VBUS), J1.B4 (VBUS), J1.B9 (VBUS)
Other:
- note removed: "FIXME"
