File: buck-converter-real.kicad_sch (KiCad schematic)
At the start: 115 parts, among them J1 USB_C_Receptacle_USB2.0_16P, J10 I2C1, J11 SWD, J12 Conn_01x04, J13 Conn_01x15, J14 Conn_01x04, J15 Conn_01x06, J4 POWER, J6 DM3CS-SF, J7 Conn_01x06, J8 I2C1, J9 SWD, Q1 CSD18540Q5B - 60-V, U1 AP2112K-3.3 (3V3 LDO), U10 TLV75733PDRV, U2 CH32V203K8T6, U4 LMR51610YDBVR, U5 LM5109BMA/NOPB, U6 TPT482-VS2R, U7 TCAN3414DDFR, U8 TPS61022, Y1 8MHz 20pF

Commit message: Remapping board, placing groups
Parts:
- R13, R16, R23, R24: footprint Resistor_SMD:R_0805_2012Metric_Pad1.20x1.40mm_HandSolder -> Resistor_SMD:R_0603_1608Metric
Other:
- moved on the sheet: C11, C20, D4
Changed lines of the file:
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@@
 	)
 	(junction
+		(at 655.32 273.05)
+		(diameter 0)
+		(color 0 0 0 0)
+	)
+	(junction
 		(at 259.08 100.33)
 		(diameter 0)
@@
 	)
 	(junction
+		(at 673.1 261.62)
+		(diameter 0)
+		(color 0 0 0 0)
+	)
+	(junction
 		(at 341.63 125.73)
 		(diameter 0)
@@
 	)
 	(junction
-		(at 652.78 261.62)
-		(diameter 0)
-		(color 0 0 0 0)
-	)
-	(junction
-		(at 673.1 273.05)
-		(diameter 0)
-		(color 0 0 0 0)
-	)
-	(junction
 		(at 533.4 279.4)
 		(diameter 0)
@@
 	)
 	(junction
-		(at 673.1 261.62)
-		(diameter 0)
-		(color 0 0 0 0)
-	)
-	(junction
 		(at 598.17 261.62)
 		(diameter 0)
@@
 	)
 	(junction
-		(at 632.46 261.62)
-		(diameter 0)
-		(color 0 0 0 0)
-	)
-	(junction
 		(at 593.09 339.09)
 		(diameter 0)
@@
 	)
 	(junction
+		(at 645.16 261.62)
+		(diameter 0)
+		(color 0 0 0 0)
+	)
+	(junction
 		(at 375.92 104.14)
 		(diameter 0)
@@
 	)
 	(junction
-		(at 652.78 273.05)
+		(at 261.62 275.59)
 		(diameter 0)
 		(color 0 0 0 0)
 	)
 	(junction
-		(at 261.62 275.59)
+		(at 533.4 287.02)
 		(diameter 0)
 		(color 0 0 0 0)
 	)
 	(junction
-		(at 533.4 287.02)
+		(at 655.32 261.62)
 		(diameter 0)
 		(color 0 0 0 0)
@@
 	)
 	(junction
+		(at 673.1 273.05)
+		(diameter 0)
+		(color 0 0 0 0)
+	)
+	(junction
 		(at 369.57 87.63)
 		(diameter 0)
@@
 	(wire
 		(pts
-			(xy 673.1 261.62) (xy 673.1 262.89)
-		)
-		(stroke
-			(width 0)
-			(type default)
-		)
-	)
-	(wire
-		(pts
 			(xy 261.62 275.59) (xy 273.05 275.59)
 		)
@@
 	(wire
 		(pts
-			(xy 623.57 261.62) (xy 632.46 261.62)
+			(xy 623.57 261.62) (xy 645.16 261.62)
 		)
 		(stroke
@@
 	(wire
 		(pts
+			(xy 645.16 270.51) (xy 645.16 273.05)
+		)
+		(stroke
+			(width 0)
+			(type default)
+		)
+	)
+	(wire
+		(pts
 			(xy 698.5 269.24) (xy 689.61 269.24)
 		)
@@
 	(wire
 		(pts
+			(xy 655.32 261.62) (xy 673.1 261.62)
+		)
+		(stroke
+			(width 0)
+			(type default)
+		)
+	)
+	(wire
+		(pts
 			(xy 598.17 339.09) (xy 593.09 339.09)
 		)
@@
 	(wire
 		(pts
+			(xy 645.16 262.89) (xy 645.16 261.62)
+		)
+		(stroke
+			(width 0)
+			(type default)
+		)
+	)
+	(wire
+		(pts
 			(xy 266.7 88.9) (xy 273.05 88.9)
 		)
@@
 	(wire
 		(pts
-			(xy 632.46 261.62) (xy 632.46 262.89)
+			(xy 655.32 261.62) (xy 655.32 262.89)
 		)
 		(stroke
@@
 	(wire
 		(pts
-			(xy 652.78 273.05) (xy 652.78 270.51)
+			(xy 673.1 273.05) (xy 673.1 270.51)
 		)
 		(stroke
@@
 	(wire
 		(pts
-			(xy 673.1 261.62) (xy 689.61 261.62)
-		)
-		(stroke
-			(width 0)
-			(type default)
-		)
-	)
-	(wire
-		(pts
 			(xy 375.92 111.76) (xy 359.41 111.76)
 		)
@@
 	(wire
 		(pts
-			(xy 652.78 261.62) (xy 673.1 261.62)
-		)
-		(stroke
-			(width 0)
-			(type default)
-		)
-	)
-	(wire
-		(pts
 			(xy 195.58 321.31) (xy 220.98 321.31)
 		)
@@
 	(wire
 		(pts
-			(xy 632.46 261.62) (xy 652.78 261.62)
-		)
-		(stroke
-			(width 0)
-			(type default)
-		)
-	)
-	(wire
-		(pts
 			(xy 215.9 156.21) (xy 215.9 162.56)
 		)
@@
 	(wire
 		(pts
-			(xy 652.78 273.05) (xy 673.1 273.05)
+			(xy 430.53 321.31) (xy 476.25 321.31)
 		)
 		(stroke
@@
 	(wire
 		(pts
-			(xy 430.53 321.31) (xy 476.25 321.31)
+			(xy 259.08 100.33) (xy 259.08 101.6)
 		)
 		(stroke
@@
 	(wire
 		(pts
-			(xy 259.08 100.33) (xy 259.08 101.6)
+			(xy 544.83 364.49) (xy 544.83 370.84)
 		)
 		(stroke
@@
 	(wire
 		(pts
-			(xy 544.83 364.49) (xy 544.83 370.84)
+			(xy 387.35 87.63) (xy 429.26 87.63)
 		)
 		(stroke
@@
 	(wire
 		(pts
-			(xy 387.35 87.63) (xy 429.26 87.63)
+			(xy 645.16 273.05) (xy 655.32 273.05)
 		)
 		(stroke
@@
 	(wire
 		(pts
-			(xy 652.78 261.62) (xy 652.78 262.89)
+			(xy 673.1 261.62) (xy 673.1 262.89)
 		)
 		(stroke
@@
 	(wire
 		(pts
-			(xy 673.1 273.05) (xy 673.1 270.51)
-		)
-		(stroke
-			(width 0)
-			(type default)
-		)
-	)
-	(wire
-		(pts
 			(xy 241.3 213.36) (xy 252.73 213.36)
 		)
@@
 	(wire
 		(pts
-			(xy 632.46 273.05) (xy 652.78 273.05)
+			(xy 655.32 273.05) (xy 673.1 273.05)
 		)
 		(stroke
@@
 	(wire
 		(pts
+			(xy 645.16 261.62) (xy 655.32 261.62)
+		)
+		(stroke
+			(width 0)
+			(type default)
+		)
+	)
+	(wire
+		(pts
 			(xy 572.77 311.15) (xy 572.77 316.23)
 		)
@@
 	(wire
 		(pts
-			(xy 632.46 273.05) (xy 632.46 270.51)
+			(xy 655.32 273.05) (xy 655.32 270.51)
 		)
 		(stroke
@@
 	(wire
 		(pts
+			(xy 673.1 261.62) (xy 689.61 261.62)
+		)
+		(stroke
+			(width 0)
+			(type default)
+		)
+	)
+	(wire
+		(pts
 			(xy 598.17 261.62) (xy 598.17 259.08)
 		)
@@
 			)
 		)
-		(property "Footprint" "Resistor_SMD:R_0805_2012Metric_Pad1.20x1.40mm_HandSolder"
+		(property "Footprint" "Resistor_SMD:R_0603_1608Metric"
 			(at 401.574 192.024 90)
 			(hide yes)
@@
 	(symbol
 		(lib_id "PCM_Diode_TVS_AKL:SMBJ36A")
-		(at 673.1 266.7 90)
+		(at 645.16 266.7 90)
 		(unit 1)
 		(body_style 1)
@@
 		(dnp no)
 		(property "Reference" "D4"
-			(at 674.37 263.652 90)
+			(at 646.43 263.652 90)
 			(show_name no)
 			(do_not_autoplace no)
@@
 		)
 		(property "Value" "SMBJ43A - 43VWM 69.4VC"
-			(at 661.162 258.318 90)
+			(at 628.396 275.082 90)
 			(show_name no)
 			(do_not_autoplace no)
@@
 		)
 		(property "Footprint" "Diode_SMD:D_SMB"
-			(at 673.1 266.7 0)
+			(at 645.16 266.7 0)
 			(hide yes)
 			(show_name no)
@@
 		)
 		(property "Datasheet" "https://www.tme.eu/Document/0b6222bec7e12d83185b51d73cb6a54d/SMBJ_ser.pdf"
-			(at 673.1 266.7 0)
+			(at 645.16 266.7 0)
 			(hide yes)
 			(show_name no)
@@
 		)
 		(property "Description" "SMB Unidirectional TVS diode, 36V, 600W, Alternate KiCAD Library"
-			(at 673.1 266.7 0)
+			(at 645.16 266.7 0)
 			(hide yes)
 			(show_name no)
@@
 			)
 		)
-		(property "Footprint" "Resistor_SMD:R_0805_2012Metric_Pad1.20x1.40mm_HandSolder"
+		(property "Footprint" "Resistor_SMD:R_0603_1608Metric"
 			(at 367.284 277.114 90)
 			(hide yes)
@@
 			)
 		)
-		(property "Footprint" "Resistor_SMD:R_0805_2012Metric_Pad1.20x1.40mm_HandSolder"
+		(property "Footprint" "Resistor_SMD:R_0603_1608Metric"
 			(at 339.344 269.494 90)
 			(hide yes)
@@
 	(symbol
 		(lib_id "PCM_Capacitor_AKL:C_1206")
-		(at 632.46 266.7 0)
+		(at 655.32 266.7 0)
 		(unit 1)
 		(body_style 1)
@@
 		(fields_autoplaced yes)
 		(property "Reference" "C11"
-			(at 636.27 265.4299 0)
+			(at 659.13 265.4299 0)
 			(show_name no)
 			(do_not_autoplace no)
@@
 		)
 		(property "Value" "1206 10uF"
-			(at 636.27 267.9699 0)
+			(at 659.13 267.9699 0)
 			(show_name no)
 			(do_not_autoplace no)
@@
 		)
 		(property "Footprint" "PCM_Capacitor_SMD_AKL:C_1206_3216Metric"
-			(at 633.4252 270.51 0)
+			(at 656.2852 270.51 0)
 			(hide yes)
 			(show_name no)
@@
 		)
 		(property "Datasheet" ""
-			(at 632.46 266.7 0)
+			(at 655.32 266.7 0)
 			(hide yes)
 			(show_name no)
@@
 		)
 		(property "Description" "SMD 1206 MLCC capacitor, Alternate KiCad Library"
-			(at 632.46 266.7 0)
+			(at 655.32 266.7 0)
 			(hide yes)
 			(show_name no)
@@
 	(symbol
 		(lib_id "PCM_Capacitor_AKL:C_1206")
-		(at 652.78 266.7 0)
+		(at 673.1 266.7 0)
 		(unit 1)
 		(body_style 1)
@@
 		(dnp no)
 		(property "Reference" "C20"
-			(at 655.828 264.16 0)
+			(at 676.148 264.16 0)
 			(show_name no)
 			(do_not_autoplace no)
@@
 		)
 		(property "Value" "1206 10uF"
-			(at 655.828 266.7 0)
+			(at 676.148 266.7 0)
 			(show_name no)
 			(do_not_autoplace no)
@@
 		)
 		(property "Footprint" "PCM_Capacitor_SMD_AKL:C_1206_3216Metric"
-			(at 653.7452 270.51 0)
+			(at 674.0652 270.51 0)
 			(hide yes)
 			(show_name no)
@@
 		)
 		(property "Datasheet" ""
-			(at 652.78 266.7 0)
+			(at 673.1 266.7 0)
 			(hide yes)
 			(show_name no)
@@
 		)
 		(property "Description" "SMD 1206 MLCC capacitor, Alternate KiCad Library"
-			(at 652.78 266.7 0)
+			(at 673.1 266.7 0)
 			(hide yes)
 			(show_name no)
@@
 			)
 		)
-		(property "Footprint" "Resistor_SMD:R_0805_2012Metric_Pad1.20x1.40mm_HandSolder"
+		(property "Footprint" "Resistor_SMD:R_0603_1608Metric"
 			(at 414.274 192.024 90)
 			(hide yes)

Commit message: Swap to 12V LDO
Parts:
- removed C39: 2.2uF, Capacitor_SMD:C_0603_1608Metric, symbol Device:C
- removed C41, C48: 100nF, Capacitor_SMD:C_0603_1608Metric, symbol Device:C
- removed C46, C47: 22uF 10V X7R/X5R 0805, Capacitor_SMD:C_0805_2012Metric_Pad1.18x1.45mm_HandSolder, symbol PCM_Capacitor_AKL:C_0805
- removed D1: BAT54C, PCM_Package_TO_SOT_SMD_AKL:SOT-23, symbol PCM_Diode_Schottky_AKL:BAT54C
- removed J13: Conn_01x15, Connector_PinSocket_2.54mm:PinSocket_1x15_P2.54mm_Vertical, symbol Connector_Generic:Conn_01x15
- removed J6: DM3CS-SF, Connector_Card:microSD_HC_Hirose_DM3D-SF, symbol 2026-05-05_06-59-55:DM3CS-SF
- removed L3: 68u, Inductor_SMD:L_Chilisin_BWVS00606020, symbol Device:L
- removed R35: 309k, Capacitor_SMD:C_0603_1608Metric, symbol Device:R_US
- removed R36: 22.1k, Capacitor_SMD:C_0603_1608Metric, symbol Device:R_US
- removed R47: 1.5m, Capacitor_SMD:C_0603_1608Metric, symbol Device:R_US
- removed R48: 100k, Capacitor_SMD:C_0603_1608Metric, symbol Device:R_US
- removed U4: LMR51610YDBVR, Package_TO_SOT_SMD:SOT-23-6, symbol Regulator_Switching:LMR51430
- added C24: 1u 100V, Capacitor_SMD:C_0805_2012Metric, symbol Device:C
- added C25: 10u 16V, Capacitor_SMD:C_0805_2012Metric, symbol Device:C
- added D7: SMAJ5.0CA clamp@9.2V, Diode_SMD:D_SMA, symbol Diode:SMAJ5.0CA
- added D8: BAT54C, Package_TO_SOT_SMD:TSOT-23, symbol Diode:BAT54W
- added J13: CAN, Connector_JST:JST_SH_BM04B-SRSS-TB_1x04-1MP_P1.00mm_Vertical, symbol Connector_Generic:Conn_01x04
- added J2: Conn_01x10, Connector_PinHeader_2.54mm:PinHeader_1x10_P2.54mm_Vertical, symbol Connector_Generic:Conn_01x10
- added J3: MSD-1-A, buck-forest:CUI_MSD-1-A, symbol MSD-1-A:MSD-1-A
- added U12: INA180A1, Package_TO_SOT_SMD:SOT-23-5, symbol Amplifier_Current:INA180A1
- added U4: ZXTR2012K-13 12V@50mA vin<100V, Package_TO_SOT_SMD:TO-252-2, symbol Regulator_Linear:AMS1117CD-2.85
- C17, C18: footprint Capacitor_SMD:C_0805_2012Metric_Pad1.18x1.45mm_HandSolder -> Capacitor_SMD:C_0603_1608Metric
- D4: value SMBJ43A - 43VWM 69.4VC -> SMBJ54A
- J1: footprint Connector_USB:USB_C_Receptacle_G-Switch_GT-USB-7010ASV -> Connector_USB:USB_C_Receptacle_GCT_USB4105-xx-A_16P_TopMnt_Horizontal
- J10: symbol Connector_Generic_Shielded:Conn_01x04_Shielded -> Connector_Generic:Conn_01x04
- J7: footprint (none) -> TerminalBlock_Phoenix:TerminalBlock_Phoenix_MPT-0,5-6-2.54_1x06_P2.54mm_Horizontal
- J9: symbol Connector_Generic:Conn_01x04 -> Connector_Generic_Shielded:Conn_01x04_Shielded
- R1: value Shunt 50m Ohm -> Shunt 50m Ohm 2512; footprint PCM_Resistor_SMD_AKL:R_2512_6332Metric -> Resistor_SMD:R_2512_6332Metric_Pad1.40x3.35mm_HandSolder; symbol PCM_Resistor_AKL:R_2512 -> Device:R_Shunt_US
- R11: value 10K -> 100K
- R15: value 1.5K -> 10k
- R25, R26: footprint Resistor_SMD:R_0805_2012Metric_Pad1.20x1.40mm_HandSolder -> Resistor_SMD:R_0603_1608Metric_Pad0.98x0.95mm_HandSolder
- R30, R31: value 4.7K -> 4.7K 0805
- R38, R39, R40: value 0 -> TBD
- RST1: footprint Button_Switch_SMD:SW_SPST_Omron_B3FS-100xP -> Button_Switch_SMD:SW_SPST_PTS647_Sx38
- SMA1: renamed from SMA-915/433MHz1; value SMA-ANT -> ANT-SMA
- U5: value LM5109BMA/NOPB -> LM5109BMA
Connections:
- net +3.3V: now also J9.3 (Pin_3), J13.4 (Pin_4), J2.3 (Pin_3), J3.4 (VDD), U12.5 (V+); no longer J9.2 (Pin_2)
- net +BATT: now also C22.1, C23.1, L2.2, R12.1
- net BAT_ISENSE: now also U12.1; no longer J15.4 (Pin_4), J15.5 (Pin_5), J15.6 (Pin_6), R1.2
- net GND: now also J7.1 (Pin_1), J9.4 (Pin_4), C24.2, C25.2, D7.1 (A1), J13.1 (Pin_1), J2.2 (Pin_2), J3.6 (VSS), J3.G1 (COVER_GND), J3.G2 (COVER_GND__1), J3.G3 (COVER_GND__2), J3.G4 (COVER_GND__3), U12.2 (GND), U4.1 (GND); no longer C22.1, C23.1, J7.6 (Pin_6), J9.1 (Pin_1), L2.2, R12.1
- net SPI-CITO: now also J3.7 (DAT0)
- net SPI-COTI: now also J3.3 (CMD)
- net SPI-CS: now also J3.2 (CD/DAT3)
- net SPI-SCK: now also J3.5 (CLK)
- net SWD-WIO-CLK: now also J9.1 (Pin_1); no longer J9.4 (Pin_4)
- net SWD-WIO-IO: now also J9.2 (Pin_2); no longer J9.3 (Pin_3)
- net Solar In: now also C24.1, U4.3 (VI)
- net VBUS: now also J2.1 (Pin_1)
- net at C44.1, R33.2, R34.2: now also J7.6 (Pin_6), D7.2 (A2); no longer J7.1 (Pin_1)
- net HS: now reaches C17.1, D3.1 (K), L2.1, Q1.1 (S), Q1.2 (S), Q1.3 (S), U5.6 (HS)
- net CAN_HI: now reaches R37.1, U7.7 (CANH)
- net CAN_HI: now also J13.3 (Pin_3)
- net CAN_TX: now reaches R45.2, U7.1 (TXD)
- net at U2.10 (PA4/ADC4): now also J2.8 (Pin_8)
- net at U2.11 (PA5/ADC5): now also J2.9 (Pin_9)
- net at U2.12 (PA6/ADC6): now also J2.10 (Pin_10)
- net CAN_S: now reaches U2.18 (PA8)
- net CAN_S: now also U7.8 (S)
- net CAN_FAULT: now reaches U2.25 (PA15)
- net CAN_FAULT: now also U7.5 (FAULT)
- net at U2.6 (PA0/WKUP/ADC0): now also J2.4 (Pin_4)
- net at U2.7 (PA1/ADC1): now also J2.5 (Pin_5)
- net at U2.8 (PA2/ADC2): now also J2.6 (Pin_6)
- net at U2.9 (PA3/ADC3): now also J2.7 (Pin_7)
- net at C17.2, U5.8 (HB): now also D8.3 (K)
- net RS422_A: now reaches J7.5 (Pin_5)
- net RS422_A: now also U6.9 (A); no longer U6.6 (Y)
- net RS422_B: now reaches J7.4 (Pin_4)
- net RS422_B: now also U6.8 (B); no longer U6.7 (Z)
- net RS422_Z: now reaches J7.3 (Pin_3)
- net RS422_Z: now also U6.7 (Z); no longer U6.8 (B)
- net RS422_Y: now reaches J7.2 (Pin_2)
- net RS422_Y: now also U6.6 (Y); no longer U6.9 (A)
- net CAN_RX: now reaches R46.2, U7.4 (RXD)
- net CAN_LOW: now reaches R44.2, U7.6 (CANL)
- net CAN_LOW: now also J13.2 (Pin_2)
- net 12V-buck renamed 12V
- net 12V: now also C25.1, D8.1 (A), U4.2 (VO)
- new net: R1.1, U12.4 (-)
- new net: R1.2, U12.3 (+)
- new net: J15.4 (Pin_4), J15.5 (Pin_5), J15.6 (Pin_6), R1.2
- no-connect marks 8 -> 9
Other:
- note added: "Battery"
- note added: "Default SMD size: 0603"
- note removed: "Default SMD size: 0603 unless otherwise marked"
- note removed: "I2C GPIO for EN?"
- moved on the sheet: C11, C17, C18, C20, C21, C22, C23, D2, D3, D4, D5, D6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
