File: Forest-Sensor-Platform.kicad_pcb (KiCad board)
At the start: 4 copper layers, 57 x 66 mm, 102 parts, among them J1 USB_C_2.0_16P, J10 I2C2, J14 Solar In, J2 Conn_01x05_Shielded, J3 MSD-1-A, J4 POWER, J6 Battery XT30, J7 Conn_01x06 2.54mm Screw Termi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, J8 I2C1, Q1 MBT3946DW1T2G, Q2 MCAC054P10Y-TP, Q3 BSS123NH6433XTMA1, SW1 WIO_RST, U1 INA181, U10 TLV75733PDRV, U11 TPS613222ADBV, U13 TPS22991CRAAR, U2 LM66200DRLR, U3 Wio-E5, STM32WLE5 Module, U6 TPT482-VS2R, U7 TPS22991CRAAR, U8 LM66200DRLR

Commit message: Fix net problems
Parts:
- C24: footprint Capacitor_SMD:C_1206_3216Metric -> Capacitor_SMD:C_0603_1608Metric
- L5: value 4.7 uH -> 2.2uH
- moved C24 53.4 mm to (89.8, 100.7), turned to 90 degrees
- moved R54 1.40 mm to (85.5, 101.0)
- moved D1 1.40 mm to (87.9, 101.0)
- moved C22 1.35 mm to (80.2, 99.1)
- moved C23 1.35 mm to (80.2, 101.8)
- moved TP6 1.04 mm to (84.2, 98.1)
- turned R1 to 0 degrees
- turned U1 to 180 degrees
Connections:
- C22 pad 1: /Buck Converter/Battery_Out -> Battery_Out
- C23 pad 1: /Buck Converter/Battery_Out -> Battery_Out
- C34 pad 1: /Forest-Sensor-Platform/Battery_Shunt_Low -> Battery_Out
- D3 pad 2: /Buck Converter/Battery_Out -> Battery_Out
- L6 pad 2: /Buck Converter/Battery_Out -> Battery_Out
- R1 pad 3: /Buck Converter/Battery_Out -> Battery_Out
- R11 pad 2: /Buck Converter/VSENSE_VIN -> VSENSE_VIN
- R12 pad 1: /Buck Converter/Battery_Out -> Battery_Out
- R12 pad 2: /Buck Converter/VSENSE_VOUT -> VSENSE_OUT
- R14 pad 1: /Buck Converter/VSENSE_VOUT -> VSENSE_OUT
- R15 pad 1: /Buck Converter/VSENSE_VIN -> VSENSE_VIN
- R36 pad 1: /Forest-Sensor-Platform/Receiver_Input_Enable -> /Forest-Sensor-Platform/Receiver_Output_Enable
- R37 pad 1: /Forest-Sensor-Platform/Receiver_Output_Enable -> /Forest-Sensor-Platform/Receiver_Input_Enable
- R38 pad 2: /Forest-Sensor-Platform/BAT_ISENSE -> BAT_ISENSE
- R39 pad 2: /Forest-Sensor-Platform/VSENSE_VOUT -> VSENSE_OUT
- R40 pad 2: /Forest-Sensor-Platform/VSENSE_VIN -> VSENSE_VIN
- U1 pad 1: /Buck Converter/BAT_ISENSE -> BAT_ISENSE
- U13 pad 1: /Forest-Sensor-Platform/Battery_Shunt_Low -> Battery_Out
- U3 pad 21: /Forest-Sensor-Platform/Receiver_Input_Enable -> /Forest-Sensor-Platform/Receiver_Output_Enable
- U3 pad 25: /Forest-Sensor-Platform/Receiver_Output_Enable -> /Forest-Sensor-Platform/Receiver_Input_Enable
- U6 pad 2: /Forest-Sensor-Platform/UART-1-TX -> /Forest-Sensor-Platform/Receiver_Input_Enable
- U6 pad 4: /Forest-Sensor-Platform/Receiver_Input_Enable -> /Forest-Sensor-Platform/UART-1-TX
Routing:
- net (no net): track 137.0 -> 0.00 mm, vias 8 -> 0
- net Battery_Out: track 0.00 -> 55.9 mm, vias 0 -> 4
- net /Forest-Sensor-Platform/Receiver_Output_Enable: track 0.00 -> 47.2 mm, vias 0 -> 2
- net /Forest-Sensor-Platform/UART-1-TX: track 0.00 -> 26.0 mm, vias 0 -> 2
- net /Forest-Sensor-Platform/Receiver_Input_Enable: track 26.0 -> 41.9 mm
- net BAT_ISENSE: track 0.00 -> 9.84 mm
- net /Forest-Sensor-Platform/BAT_ISENSE: track 9.64 -> 0.00 mm
- net Net-(F1-Pad1): track 37.5 -> 32.4 mm
- net /Forest-Sensor-Platform/VSENSE_VOUT: track 3.65 -> 0.00 mm
- net VSENSE_VIN: track 0.00 -> 3.48 mm
- net /Forest-Sensor-Platform/VSENSE_VIN: track 3.48 -> 0.00 mm
- net VSENSE_OUT: track 0.00 -> 3.33 mm
- net Net-(U1-+): track 4.51 -> 7.45 mm
- net Net-(U1--): track 4.51 -> 7.17 mm
- net Net-(D1-A): track 3.76 -> 5.64 mm
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