File: Forest-Sensor-Platform.kicad_pcb (KiCad board)
At the start: 4 copper layers, 57 x 66 mm, 102 parts, among them J1 USB_C_2.0_16P, J10 I2C2, J14 Solar In, J2 Conn_01x05_Shielded, J3 MSD-1-A, J4 POWER, J6 Battery XT30, J7 Conn_01x06 2.54mm Screw Termi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, J8 I2C1, Q1 MBT3946DW1T2G, Q2 MCAC054P10Y-TP, Q3 BSS123NH6433XTMA1, SW1 WIO_RST, U1 INA181, U10 TLV75733PDRV, U11 TPS613222ADBV, U13 TPS22991CRAAR, U2 LM66200DRLR, U3 Wio-E5, STM32WLE5 Module, U6 TPT482-VS2R, U7 TPS22991CRAAR, U8 LM66200DRLR

Commit message: Fix DRC errors
Parts:
- C11, C20: value 10uF 50V 1206 -> 10uF 50V
- C13, C9: value 10uF 50V -> 10uF 25V
- C16, C19, C21, C32: value 100n -> 100nF 50V
- C24: value 1 uF 50V -> 1uF 50V
- C30, C34: value 1u -> 1uF 25V
- C31, C35: value 10u -> 10uF 25V
- C46: value 22uF 10V -> 22uF 16V
- D5, D8: value SS56 60V 700mV@5A -> SK56A 60V 5A SMA
- R15, R57: value 10k -> 10K
- R21, R22, R31, R36, R37, R44: value 1m -> 1M
- R33: value DNP -> 0
- R38, R39, R40: value TBD -> 1K
- R54: value 4.7k 1206 -> 4.7K
- R55: value 100k -> 100K
- R56: value 22 -> 22R
- R58: value 2.2k -> 2.2K
- U1: value INA181 -> INA181A1
- U4: value ~ -> CH572D Module
- moved R18 0.25 mm to (103.2, 86.2)
Connections:
- J10 pad MP: (no net) -> unconnected-(J10-MountPin-PadMP)_1
- J2 pad MP: (no net) -> unconnected-(J2-MountPin-PadMP)
- J8 pad MP: (no net) -> unconnected-(J8-MountPin-PadMP)
- U10 pad 7: (no net) -> GND
- U8 pad 6: /Forest-Sensor-Platform/Batt_Out -> Battery_Out
