File: Forest-Sensor-Platform.kicad_pcb (KiCad board)
At the start: 4 copper layers, 57 x 66 mm, 114 parts, among them J1 USB_C_2.0_16P, J10 I2C2, J14 Solar In, J2 Conn_01x05_Shielded, J3 MSD-1-A, J4 POWER, J6 Battery XT30, J7 Conn_01x06 2.54mm Screw Termi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, J8 I2C1, J9 U.FL, Q1 MBT3946DW1T2G, Q2 MCAC054P10Y-TP, Q3 BSS123NH6433XTMA1, SW1 WIO_RST, U1 INA181A1, U10 TLV75733PDRV, U11 TPS613222ADBV, U13 TPS22991CRAAR, U2 LM66200DRLR, U3 Wio-E5, STM32WLE5 Module, U6 TPT482-VS2R, U7 TPS22991CRAAR, U8 LM66200DRLR, U9 CH572D, Y2 Crystal_GND2

Commit message: V1 final
Parts:
- added TP7: TestPoint, buck-forest:Testpad, B.Cu at (122.7, 121.6)
- added TP9: TestPoint, buck-forest:Testpad, B.Cu at (122.7, 119.1)
Routing:
- net /USB/CH_USR_BTN: track 0.00 -> 5.21 mm, vias 0 -> 1
- net /USB/CH_GPIO: track 0.00 -> 4.22 mm, vias 0 -> 1
- net Net-(J6-Pin_1): track 4.29 -> 5.09 mm
- net /Buck Converter/Solar In: track 56.9 -> 57.5 mm
- net GND: vias 713 -> 742
Other:
- board text added: "EN USB"
- board text added: "RS422"
- board text added: "TMPK"
