File: gps-radio-board/gps-radio-board.kicad_pcb (KiCad board)
At the start: 4 copper layers, 25 x 54 mm, 63 parts, among them J1 SMA, J2 SMA, J3 USB_C_Receptacle_USB2.0_16P, J4 JST_BATT, J5 Conn_01x04, J6 Conn_01x04, J7 Conn_01x04, J8 DM3CS-SF, U1 ESP32-C6-MINI-1U-H4, U3 SiP32431DR3, U4 AP2112K-3.3, U5 MAX-M10N, U6 MCP73831, U7 AP2112K-3.3

Commit message: Minor adjustment
Connections:
- net /I2C-2-SCA renamed /I2C-2-SDA
- U2 pad 28: +3V3 -> unconnected-(U2-VDD-Pad28)
Routing:
- net +3V3: track 35.7 -> 29.1 mm, vias 14 -> 10
- net unconnected-(U2-VDD-Pad28): track 0.00 -> 1.01 mm
Changed lines of the file:
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@@
 			(layers "F.Cu" "F.Mask" "F.Paste")
 			(roundrect_rratio 0.25)
-			(net "/I2C-2-SCA")
+			(net "/I2C-2-SDA")
 			(pinfunction "Pin_3_3")
 			(pintype "passive")
@@
 			(size 1 2.3)
 			(layers "F.Cu" "F.Mask" "F.Paste")
-			(net "/I2C-2-SCA")
+			(net "/I2C-2-SDA")
 			(pinfunction "PC1_12")
 			(pintype "input")
@@
 			(size 1 2.3)
 			(layers "F.Cu" "F.Mask" "F.Paste")
-			(net "+3V3")
+			(net "unconnected-(U2-VDD-Pad28)")
 			(pinfunction "VDD_28")
-			(pintype "input")
+			(pintype "input+no_connect")
 		)
 		(embedded_fonts no)
@@
 	)
 	(segment
-		(start 107.95 94.15)
-		(end 107.95 93.875)
-		(width 0.2)
-		(layer "F.Cu")
-		(net "+BATT")
-	)
-	(segment
 		(start 106 93.375)
 		(end 106 94.426471)
@@
 	)
 	(segment
-		(start 107.125 94.6)
-		(end 107.5 94.6)
+		(start 107.95 94.275)
+		(end 107.95 93.875)
 		(width 0.2)
 		(layer "F.Cu")
@@
 	)
 	(segment
-		(start 107.5 94.6)
-		(end 107.95 94.15)
+		(start 106 94.426471)
+		(end 106.173529 94.6)
 		(width 0.2)
 		(layer "F.Cu")
@@
 	)
 	(segment
-		(start 106 94.426471)
-		(end 106.173529 94.6)
+		(start 107.125 94.6)
+		(end 107.625 94.6)
 		(width 0.2)
 		(layer "F.Cu")
@@
 		(net "+BATT")
 	)
+	(segment
+		(start 107.625 94.6)
+		(end 107.95 94.275)
+		(width 0.2)
+		(layer "F.Cu")
+		(net "+BATT")
+	)
 	(via
 		(at 107.375 95.35)
@@
 	)
 	(segment
-		(start 109.8 110.208677)
-		(end 111.316323 110.208677)
-		(width 0.2)
-		(layer "F.Cu")
-		(net "+3V3")
-	)
-	(segment
 		(start 108.166323 107.958677)
 		(end 107.55 107.958677)
@@
 	)
 	(segment
-		(start 109.825 109.175)
-		(end 109.825 109.4)
-		(width 0.2)
-		(layer "F.Cu")
-		(net "+3V3")
-	)
-	(segment
-		(start 108.575 109.15)
-		(end 108.575 109.175)
-		(width 0.2)
-		(layer "F.Cu")
-		(net "+3V3")
-	)
-	(segment
-		(start 109.8 109.425)
-		(end 109.8 110.208677)
-		(width 0.2)
-		(layer "F.Cu")
-		(net "+3V3")
-	)
-	(segment
 		(start 91.35 115.009602)
 		(end 91.350961 115.008641)
@@
 	)
 	(segment
-		(start 109.8 110.208677)
-		(end 108.791323 110.208677)
-		(width 0.2)
-		(layer "F.Cu")
-		(net "+3V3")
-	)
-	(segment
 		(start 91.350961 115.008641)
 		(end 91.350961 116.174039)
@@
 	)
 	(segment
-		(start 108.325 109.425)
-		(end 108.325 110.042354)
-		(width 0.2)
-		(layer "F.Cu")
-		(net "+3V3")
-	)
-	(segment
 		(start 100.025 89.375)
 		(end 100.025 88.8)
@@
 	)
 	(segment
-		(start 108.575 109.15)
-		(end 108.525 109.2)
-		(width 0.2)
-		(layer "F.Cu")
-		(net "+3V3")
-	)
-	(segment
-		(start 109.825 109.4)
-		(end 109.8 109.425)
-		(width 0.2)
-		(layer "F.Cu")
-		(net "+3V3")
-	)
-	(segment
 		(start 91.350961 116.174039)
 		(end 91.35 116.175)
@@
 	)
 	(segment
-		(start 108.35 110.35)
-		(end 108.491323 110.208677)
-		(width 0.2)
-		(layer "F.Cu")
-		(net "+3V3")
-	)
-	(segment
-		(start 108.325 110.042354)
-		(end 108.491323 110.208677)
-		(width 0.2)
-		(layer "F.Cu")
-		(net "+3V3")
-	)
-	(segment
-		(start 108.35 110.558675)
-		(end 108.35 110.35)
-		(width 0.2)
-		(layer "F.Cu")
-		(net "+3V3")
-	)
-	(segment
 		(start 111.15 105.7)
 		(end 111.15 106.4625)
@@
 	)
 	(segment
-		(start 108.575 109.175)
-		(end 108.325 109.425)
-		(width 0.2)
-		(layer "F.Cu")
-		(net "+3V3")
-	)
-	(segment
-		(start 111.316323 110.208677)
-		(end 111.325 110.2)
-		(width 0.2)
-		(layer "F.Cu")
-		(net "+3V3")
-	)
-	(segment
 		(start 111.15 106.4625)
 		(end 109.6625 106.4625)
@@
 	)
 	(segment
-		(start 108.491323 110.208677)
-		(end 109.8 110.208677)
-		(width 0.2)
-		(layer "F.Cu")
-		(net "+3V3")
-	)
-	(segment
 		(start 107.55 106.225)
 		(end 107.55 107.958677)
@@
 	)
 	(via
-		(at 111.325 110.2)
-		(size 0.6)
-		(drill 0.3)
-		(layers "F.Cu" "B.Cu")
-		(net "+3V3")
-	)
-	(via
 		(at 98.95 88.825)
 		(size 0.6)
@@
 	)
 	(via
-		(at 108.35 110.558675)
-		(size 0.6)
-		(drill 0.3)
-		(layers "F.Cu" "B.Cu")
-		(net "+3V3")
-	)
-	(via
-		(at 109.825 109.175)
-		(size 0.6)
-		(drill 0.3)
-		(layers "F.Cu" "B.Cu")
-		(net "+3V3")
-	)
-	(via
 		(at 107.55 106.225)
 		(size 0.6)
@@
 	)
 	(via
-		(at 108.575 109.15)
-		(size 0.6)
-		(drill 0.3)
-		(layers "F.Cu" "B.Cu")
-		(net "+3V3")
-	)
-	(via
 		(at 91.35 119.3)
 		(size 0.6)
@@
 		(width 0.2)
 		(layer "F.Cu")
-		(net "/I2C-2-SCA")
+		(net "/I2C-2-SDA")
 	)
 	(segment
@@
 		(width 0.2)
 		(layer "F.Cu")
-		(net "/I2C-2-SCA")
+		(net "/I2C-2-SDA")
 	)
 	(segment
@@
 		(width 0.2)
 		(layer "F.Cu")
-		(net "/I2C-2-SCA")
+		(net "/I2C-2-SDA")
 	)
 	(segment
@@
 		(width 0.2)
 		(layer "F.Cu")
-		(net "/I2C-2-SCA")
+		(net "/I2C-2-SDA")
 	)
 	(segment
@@
 		(width 0.2)
 		(layer "F.Cu")
-		(net "/I2C-2-SCA")
+		(net "/I2C-2-SDA")
 	)
 	(segment
@@
 		(width 0.2)
 		(layer "F.Cu")
-		(net "/I2C-2-SCA")
+		(net "/I2C-2-SDA")
 	)
 	(segment
@@
 		(width 0.2)
 		(layer "F.Cu")
-		(net "/I2C-2-SCA")
+		(net "/I2C-2-SDA")
 	)
 	(segment
@@
 	)
 	(segment
+		(start 109.8 110.208677)
+		(end 108.791323 110.208677)
+		(width 0.2)
+		(layer "F.Cu")
+		(net "unconnected-(U2-VDD-Pad28)")
+	)
+	(segment
