File: gps-radio-board/gps-radio-board.kicad_sch (KiCad schematic)
At the start: 63 parts, among them J1 SMA, J2 SMA, J3 USB_C_Receptacle_USB2.0_16P, J4 JST_BATT, J5 Conn_01x04, J6 Conn_01x04, J7 Conn_01x04, J8 DM3CS-SF, U1 ESP32-C6-MINI-1U-H4, U3 SiP32431DR3, U4 AP2112K-3.3, U5 MAX-M10N, U6 MCP73831, U7 AP2112K-3.3

Commit message: Minor adjustment
Connections:
- net +3V3: no longer U2.28 (VDD)
- net I2C-2-SCA renamed I2C-2-SDA
- no-connect marks 24 -> 25
Changed lines of the file:
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@@
 	)
 	(junction
-		(at 344.17 172.72)
-		(diameter 0)
-		(color 0 0 0 0)
-	)
-	(junction
 		(at 264.16 132.08)
 		(diameter 0)
@@
 	)
 	(no_connect
+		(at 340.36 172.72)
+	)
+	(no_connect
 		(at 388.62 99.06)
 	)
@@
 	(wire
 		(pts
-			(xy 340.36 172.72) (xy 344.17 172.72)
-		)
-		(stroke
-			(width 0)
-			(type default)
-		)
-	)
-	(wire
-		(pts
 			(xy 383.54 92.71) (xy 383.54 99.06)
 		)
@@
 		)
 	)
-	(label "I2C-2-SCA"
+	(label "I2C-2-SDA"
 		(at 368.3 198.12 180)
 		(effects
@@
 		(dnp no)
 		(property "Reference" "J5"
-			(at 287.274 244.348 0)
+			(at 291.338 242.57 0)
 			(show_name no)
 			(do_not_autoplace no)
@@
 		)
 		(property "Value" "Conn_01x04"
-			(at 287.274 242.062 0)
+			(at 289.56 226.822 0)
 			(show_name no)
 			(do_not_autoplace no)
